Commit message: updated the urdf to rotate the gripper; remove the geometry of the virtual_ee_link in limited urdf

File: ur_e_description/urdf/ur5e_cam_2f85_joint_limited_robot.urdf.xacro (robot description, xacro)
@@ -45,7 +45,7 @@
     <parent link="robotiq_cam_link" />
     <child link = "robotiq_arg2f_base_link" />
-    <origin xyz="0.0 0.0 0.0112" rpy="0.0 0.0 0.0" />
+    <origin xyz="0.0 0.0 0.0112" rpy="0.0 0.0 ${pi / 2.0}" />
   </joint>
-  <link name="virtual_ee_link">
+<!--   <link name="virtual_ee_link">
       <visual>
         <origin xyz="0 0 0" rpy="0 0 0" />
@@ -57,5 +57,6 @@
         </material>
       </visual>
-  </link>
+  </link> -->
+  <link name="virtual_ee_link" />
   <joint name="virtual_ee_joint" type="fixed">
     <parent link="robotiq_arg2f_base_link" />

File: ur_e_description/urdf/ur5e_cam_2f85_robot.urdf.xacro (robot description, xacro)
@@ -30,5 +30,5 @@
     <parent link="robotiq_cam_link" />
     <child link = "robotiq_arg2f_base_link" />
-    <origin xyz="0.0 0.0 0.0112" rpy="0.0 0.0 0.0" />
+    <origin xyz="0.0 0.0 0.0112" rpy="0.0 0.0 ${pi / 2.0}" />
   </joint>
 <!--   <link name="virtual_ee_link">
@@ -43,10 +43,15 @@
       </visual>
   </link> -->
-  <link name="virtual_ee_link" />
+<!--   <link name="virtual_ee_link" />
   <joint name="virtual_ee_joint" type="fixed">
     <parent link="tool0" />
     <child link = "virtual_ee_link" />
     <origin xyz="0.0 0.0 0.1654" rpy="0.0 0.0 0.0" />
-    <!-- <origin xyz="0.0 0.0 0.1445" rpy="0.0 0.0 0.0" /> -->
+  </joint> -->
+  <link name="virtual_ee_link" />
+  <joint name="virtual_ee_joint" type="fixed">
+    <parent link="robotiq_arg2f_base_link" />
+    <child link = "virtual_ee_link" />
+    <origin xyz="0.0 0.0 0.1445" rpy="0.0 0.0 0.0" />
   </joint>
 </robot>
